Commit message: 目前已经解决了抽搐问题，urdf中base_link和pelvis的角度关节设置有误导致的，但目前还是没有有效的运动

File: src/ros_navigation_humanoid/robot_descriptions/unitree_g1/g1_29dof_with_hand copy.urdf (robot description, URDF)
Before this commit: robot g1_29dof_with_hand, 57 links, 56 joints
Links:
- link base_link: mass None -> 3.813
- link pelvis: mass 3.813 -> None
Joints:
- removed joint odom_to_base_link
- added joint base_to_pelvis: type fixed, parent base_link, child pelvis, origin xyz=0 0 0.8 rpy=0 0 0
- joint floating_base_joint: child pelvis -> base_link; origin xyz=0 0 0.8 rpy=0 0 0 -> xyz=0 0 0 rpy=0 0 0; parent base_link -> odom; type fixed -> continuous
