Commit message: 0806暂存，增加激光雷达，目前机器人一直在原地转圈，暂时无法解决

File: src/ros_navigation_humanoid/robot_descriptions/unitree_g1/g1_29dof_with_hand_0801.urdf (robot description, URDF)
Before this commit: robot g1_29dof_with_hand, 58 links, 57 joints
Links:
- removed link laser_link
Joints:
- removed joint laser_joint
