Commit message: 0723暂存：增加2d雷达节点，修复tf变换由map->odom->plevis

File: src/ros_navigation_humanoid/robot_descriptions/unitree_g1/g1_29dof_with_hand.urdf (robot description, URDF)
Before this commit: robot g1_29dof_with_hand, 55 links, 54 joints
Links:
- added link odom, mass 0.001
Joints:
- added joint map_to_odom: type fixed, parent map, child odom, origin xyz=0 0 0 rpy=0 0 0
- joint floating_base_joint: parent map -> odom; type fixed -> floating

Commit message: 修正tf变换:map->odom->base_link->pelvis；修复控制器和代价地图订阅不到激光的问题；目前全链路已经打通，已经有角速度，但无线速度，继续排查

File: src/ros_navigation_humanoid/robot_descriptions/unitree_g1/g1_29dof_with_hand.urdf (robot description, URDF)
Before this commit: robot g1_29dof_with_hand, 56 links, 55 joints
Links:
- added link base_link, mass 3.813
- link pelvis: mass 3.813 -> None
Joints:
- added joint base_to_pelvis: type fixed, parent base_link, child pelvis, origin xyz=0 0 0 rpy=0 0 0
- joint floating_base_joint: child pelvis -> base_link; origin (none) -> xyz=0 0 0.8 rpy=0 0 0; type floating -> continuous

Commit message: 目前已经激光已经可以转动了，但机器人的身体只会转动和抽搐，线速度还没有，角速度有

File: src/ros_navigation_humanoid/robot_descriptions/unitree_g1/g1_29dof_with_hand.urdf (robot description, URDF)
Before this commit: robot g1_29dof_with_hand, 57 links, 56 joints
Joints:
- joint base_to_pelvis: origin xyz=0 0 0 rpy=0 0 0 -> xyz=0 0 0.8 rpy=0 0 0
- joint floating_base_joint: origin xyz=0 0 0.8 rpy=0 0 0 -> xyz=0 0 0 rpy=0 0 0

Commit message: 0808暂存，增加mapping和navigation代码，基本上能正常运动，但是范围很小，速度很慢

File: src/ros_navigation_humanoid/robot_descriptions/unitree_g1/g1_29dof_with_hand.urdf (robot description, URDF)
Before this commit: robot g1_29dof_with_hand, 58 links, 57 joints
Joints:
- joint laser_joint: origin xyz=0 0 0.56 rpy=0 0 0 -> xyz=0 0 0.425 rpy=0 0 0
